File: hardware/modules/MCU/V3/MCU_M_V3.kicad_pcb (KiCad board)
At the start: 4 copper layers, 26.9 x 19 mm, 21 parts, among them Q1 IRLML6246TRPBF, U1 STM32F405OGYx, U2 STULPI01B, Y1 NX3225GA-10.000M-STD-CRG-2, Y3 FX135A-327

Commit message: MCU_V3_SCH added
Parts:
- removed D2: 1SS417CT,L3F, SamacSys_Parts:1SS417CTL3F
- added C21: GRM155Z71A105KE01J, SamacSys_Parts:CAPC1005X55N, F.Cu at (176.3, 93.0)
- added C22: GRM155Z71A105KE01J, SamacSys_Parts:CAPC1005X55N, F.Cu at (179.6, 94.4)
- added C23: GRM155Z71A105KE01J, SamacSys_Parts:CAPC1005X55N, F.Cu at (175.5, 95.6)
- added C24: GRM155Z71A105KE01J, SamacSys_Parts:CAPC1005X55N, F.Cu at (172.7, 95.6)
- added J1: M50-3530242, SamacSys_Parts:HDRV2W40P0X127_1X2_254X210X420P, F.Cu at (172.2, 97.6)
- added J2: M50-3530342, SamacSys_Parts:HDRV3W40P0X127_1X3_381X210X430P, F.Cu at (173.3, 101.8)
- added R11: ERJ-3EKF1002V, SamacSys_Parts:ERJ3EK_(0603), F.Cu at (179.5, 98.6)
- added R12: ERJ-3EKF1002V, SamacSys_Parts:ERJ3EK_(0603), F.Cu at (180.8, 99.9)
- added R21: RK73Z1ETTP, SamacSys_Parts:RESC1005X40N, F.Cu at (175.7, 99.5)
- added R22: RK73Z1ETTP, SamacSys_Parts:RESC1005X40N, F.Cu at (172.3, 99.5)
- added R23: ERA2AED123X, SamacSys_Parts:ERA2AED122X, F.Cu at (173.2, 93.2)
- added R24: RK73Z1ETTP, SamacSys_Parts:RESC1005X40N, F.Cu at (186.7, 101.8)
- added R25: RK73Z1ETTP, SamacSys_Parts:RESC1005X40N, F.Cu at (183.3, 101.8)
- added R26: RK73Z1ETTP, SamacSys_Parts:RESC1005X40N, F.Cu at (180.4, 101.9)
- added R27: RK73Z1ETTP, SamacSys_Parts:RESC1005X40N, F.Cu at (183.3, 99.6)
- added R28: RK73Z1ETTP, SamacSys_Parts:RESC1005X40N, F.Cu at (186.7, 99.6)
- added R4: CPF0603F100KC1, SamacSys_Parts:RESC1608X55N, F.Cu at (177.3, 91.2)
- D1: value 1SS417CT,L3F -> BAT54S; footprint SamacSys_Parts:1SS417CTL3F -> Package_TO_SOT_SMD:SOT-23
- moved D1 6.17 mm to (179.2, 88.9)
- moved C1 1.32 mm to (174.7, 91.2)
- moved R1 0.20 mm to (176.6, 88.7)
- renumbered Y1 to Y11, Y3 to Y12
Connections:
- C101 pad 1: /GND -> GND
- C102 pad 1: /GND -> GND
- C103 pad 1: /GND -> GND
- C12 pad 1: /GND -> GND
- C13 pad 2: /GND -> GND
- C14 pad 1: /GND -> GND
- C15 pad 2: /GND -> GND
- D1 pad 1: /+3.3 -> GND
- D1 pad 2: /MCU_BOOT0 -> /+3.3
- H1 pad 1: /+5 -> /+3.3
- H1 pad 14: /GND -> GND
- H1 pad 2: /+3.3 -> /VCC3
- H1 pad 8: /GND -> GND
- H2 pad 12: /GND -> GND
- H2 pad 18: /GND -> GND
- Q1 pad 2: /GND -> GND
- R3 pad 2: /GND -> GND
- U1 pad A2: unconnected-(U1-PadA2) -> /SW_CLK
- U1 pad A3: unconnected-(U1-PadA3) -> /PC12
- U1 pad A5: unconnected-(U1-PadA5) -> /M2_D4
- U1 pad A6: unconnected-(U1-PadA6) -> /B5
- U1 pad B4: unconnected-(U1-PadB4) -> /PD2
- U1 pad B5: unconnected-(U1-PadB5) -> /M2_D3
- U1 pad B6: unconnected-(U1-PadB6) -> /B3
- U1 pad B7: unconnected-(U1-PadB7) -> /B2
- U1 pad C1: unconnected-(U1-PadC1) -> /PA11
- U1 pad C10: unconnected-(U1-PadC10) -> /M4_D4
- U1 pad C2: unconnected-(U1-PadC2) -> /PA12
- U1 pad C4: unconnected-(U1-PadC4) -> /M3_D2
- U1 pad C7: unconnected-(U1-PadC7) -> /B1
- U1 pad C8: unconnected-(U1-PadC8) -> /P0_D1
- U1 pad C9: /GND -> GND
- U1 pad D1: unconnected-(U1-PadD1) -> /M2_D5
- U1 pad D2: unconnected-(U1-PadD2) -> /M4_D1
- U1 pad D3: unconnected-(U1-PadD3) -> /M4_D2
- U1 pad D4: unconnected-(U1-PadD4) -> /SW_IO
- U1 pad D5: unconnected-(U1-PadD5) -> /M3_D1
- U1 pad D8: unconnected-(U1-PadD8) -> /P0_D2
- U1 pad D9: /GND -> GND
- U1 pad E1: unconnected-(U1-PadE1) -> /P0_D3
- U1 pad E2: unconnected-(U1-PadE2) -> /M4_D6
- U1 pad E5: /GND -> GND
- U1 pad E7: /GND -> GND
- U1 pad E8: /GND -> GND
- U1 pad F1: unconnected-(U1-PadF1) -> /ULPI_RST
- U1 pad F2: unconnected-(U1-PadF2) -> /ULPI_PWRDN
- U1 pad F3: unconnected-(U1-PadF3) -> /M1_D7
- U1 pad F5: unconnected-(U1-PadF5) -> /M1_D5
- U1 pad F8: unconnected-(U1-PadF8) -> /M2_D1
- U1 pad G1: unconnected-(U1-PadG1) -> /M2_D9
- U1 pad G2: unconnected-(U1-PadG2) -> /M2_D10
- U1 pad G3: unconnected-(U1-PadG3) -> /M2_D8
- U1 pad G4: unconnected-(U1-PadG4) -> /M1_D6
- U1 pad G5: unconnected-(U1-PadG5) -> /M1_D3
- U1 pad H1: unconnected-(U1-PadH1) -> /M3_D7
- U1 pad H10: /GND -> GND
- U1 pad H2: unconnected-(U1-PadH2) -> /M2_D6
- U1 pad H3: unconnected-(U1-PadH3) -> /M2_D7
- U1 pad H8: unconnected-(U1-PadH8) -> /M1_D4
- U1 pad J10: unconnected-(U1-PadJ10) -> /M2_D2
- U1 pad J2: unconnected-(U1-PadJ2) -> /M4_D7
- U1 pad J7: /GND -> GND
- U1 pad J8: unconnected-(U1-PadJ8) -> /B4
- U1 pad J9: unconnected-(U1-PadJ9) -> /M4_D3
- U2 pad B2: Net-(U2-PadB2) -> /+3.3
- U2 pad B3: Net-(U2-PadB2) -> /+3.3
- U2 pad B4: /GND -> GND
- U2 pad B5: Net-(U2-PadB2) -> /+3.3
- U2 pad C1: unconnected-(U2-PadC1) -> Net-(R26-Pad2)
- U2 pad C2: unconnected-(U2-PadC2) -> Net-(U2-PadC2)
- U2 pad C3: /GND -> /ULPI_PWRDN
- U2 pad C4: /+3.3 -> /ULPI_RST
- U2 pad C5: /GND -> GND
- U2 pad D1: unconnected-(U2-PadD1) -> Net-(R25-Pad2)
- U2 pad D2: /GND -> GND
- U2 pad D3: unconnected-(U2-PadD3) -> Net-(U2-PadD3)
- U2 pad E1: /GND -> GND
- U2 pad E2: unconnected-(U2-PadE2) -> GND
- U2 pad E3: unconnected-(U2-PadE3) -> Net-(U2-PadE3)
- U2 pad E4: /GND -> GND
- U2 pad E6: unconnected-(U2-PadE6) -> Net-(U2-PadE6)
- U2 pad F3: unconnected-(U2-PadF3) -> /+3.3
- Y11 pad 2: /GND -> GND
- Y11 pad 4: /GND -> GND
Routing:
- net GND: track 0.00 -> 32.9 mm
- net /GND: track 32.9 -> 0.00 mm
- net /+3.3: track 28.4 -> 10.4 mm

Commit message: MCU_V3 draft added
Parts:
- removed C101: GMD155R71C104KA11D, SamacSys_Parts:CAPC1005X55N
- moved C21 19.8 mm to (196.1, 94.1), turned to -90 degrees
- moved R23 19.8 mm to (192.3, 98.2)
- moved C23 17.6 mm to (192.5, 91.1)
- moved C24 16.6 mm to (188.9, 92.0)
- moved C22 16.5 mm to (196.1, 96.1)
- moved C102 14.6 mm to (181.8, 96.1), turned to -90 degrees
- moved C15 11.9 mm to (178.3, 95.6), turned to -90 degrees
- moved R28 10.4 mm to (176.4, 101.2), turned to 90 degrees
- moved C103 9.21 mm to (192.5, 92.0), turned to 180 degrees
- moved U2 9.00 mm to (192.9, 95.1), turned to 90 degrees
- moved C14 8.59 mm to (178.3, 92.6), turned to -90 degrees
- moved R27 8.53 mm to (174.8, 100.6), turned to 90 degrees
- moved R24 8.46 mm to (194.3, 98.2), turned to 180 degrees
- moved Y12 7.85 mm to (180.1, 94.1), turned to -90 degrees
- moved U1 7.20 mm to (185.1, 95.1), turned to 90 degrees
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Connections:
- J1 pad 1: /VBAT -> GND
- J1 pad 2: GND -> /VBAT
- J2 pad 1: /SW_IO -> GND
- J2 pad 3: GND -> /SW_IO
Routing:
- net GND: track 32.9 -> 124.9 mm, vias 0 -> 12
- net /+3.3: track 10.4 -> 68.1 mm, vias 0 -> 12
- net /M1_D6: track 0.00 -> 24.3 mm, vias 0 -> 2
- net /M2_D10: track 0.00 -> 21.9 mm, vias 0 -> 1
- net /M2_D9: track 0.00 -> 21.8 mm, vias 0 -> 1
- net /M2_D7: track 0.00 -> 21.7 mm, vias 0 -> 2
- net /M2_D6: track 0.00 -> 20.5 mm, vias 0 -> 1
- net /M1_D4: track 0.00 -> 19.4 mm, vias 0 -> 1
- net /M1_D5: track 0.00 -> 19.1 mm, vias 0 -> 1
- net /MCU_RESET: track 0.00 -> 19.0 mm, vias 0 -> 5
- net /M2_D8: track 0.00 -> 18.8 mm, vias 0 -> 3
- net /M4_D6: track 0.00 -> 18.8 mm, vias 0 -> 2
- net /P0_D2: track 0.00 -> 18.5 mm, vias 0 -> 1
- net /P0_D1: track 0.00 -> 17.7 mm, vias 0 -> 1
- net Net-(R25-Pad2): track 0.00 -> 17.3 mm
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- removed copper zone on B.Cu, net (none)

Commit message: MCU_V3 fix1
Parts:
- moved C12 0.10 mm to (183.2, 90.0)
- moved C13 0.09 mm to (188.0, 90.0)
Routing:
- net GND: track 124.9 -> 122.1 mm
- net /+3.3: track 68.1 -> 68.9 mm

Commit message: MCU_V3 fix2
Routing:
- net /+3.3: track 68.9 -> 62.3 mm, vias 12 -> 9
- net GND: track 122.1 -> 116.5 mm
- net /M2_D1: track 16.6 -> 19.2 mm
- net /M2_D2: track 13.2 -> 15.8 mm
- net Net-(C11-Pad1): track 3.19 -> 0.62 mm
- net /M2_D8: track 18.8 -> 20.8 mm
- net /ULPI_XI: track 11.2 -> 9.64 mm
- net Net-(R25-Pad2): track 17.3 -> 15.8 mm
- net Net-(U2-PadE3): track 2.52 -> 1.23 mm
- net /ULPI_D6: track 7.30 -> 6.06 mm
- net Net-(C12-Pad2): track 4.67 -> 3.83 mm
- net Net-(C15-Pad1): track 6.74 -> 6.01 mm
- net /B4: track 14.4 -> 15.1 mm
- net /M1_D5: track 19.1 -> 18.4 mm
- net /SW_CLK: track 13.4 -> 12.7 mm
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
Commit message: MCU_V3 fix3
Parts:
- added C104: GMD155R71C104KA11D, SamacSys_Parts:CAPC1005X55N, F.Cu at (181.7, 91.5)
- moved C102 4.10 mm to (185.0, 98.6), turned to 0 degrees
- moved C11 1.82 mm to (182.6, 98.6)
- moved C15 0.51 mm to (178.5, 95.1), turned to 90 degrees
- moved C14 0.48 mm to (178.5, 93.1), turned to 90 degrees
- moved C24 0.42 mm to (188.5, 92.0), turned to 90 degrees
- moved R23 0.23 mm to (192.5, 98.3)
Connections:
- net /VCC3 renamed /+5
Routing:
- net GND: track 116.5 -> 157.4 mm, vias 12 -> 17
- net /P0_D2: track 18.5 -> 38.6 mm, vias 1 -> 2
- net /M4_D1: track 13.7 -> 33.7 mm, vias 2 -> 3
- net /P0_D1: track 17.7 -> 34.4 mm, vias 1 -> 2
- net /+3.3: track 62.3 -> 74.3 mm, vias 9 -> 18
- net /M4_D2: track 12.8 -> 22.4 mm
- net /ULPI_D7: track 8.98 -> 18.4 mm, vias 2 -> 5
- net /M2_D9: track 21.8 -> 30.4 mm
- net /M4_D6: track 18.9 -> 27.3 mm, vias 2 -> 3
- net /M2_D10: track 22.3 -> 30.6 mm
- net /M2_D4: track 11.4 -> 19.6 mm, vias 1 -> 2
- net /ULPI_XI: track 9.64 -> 17.7 mm, vias 2 -> 4
- net /M1_D7: track 13.2 -> 20.2 mm
- net /M1_D3: track 16.7 -> 23.3 mm, vias 1 -> 3
- net /B5: track 10.0 -> 16.2 mm
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- added copper zone on B.Cu, net GND
- added copper zone on F.Cu, net GND

Commit message: MCU_V3 fix4
Routing:
- net /+5: track 0.00 -> 27.4 mm, vias 0 -> 1
- net GND: track 157.4 -> 165.9 mm, vias 17 -> 23
