File: hardware/modules/MCU/V3/MCU_M_V3.kicad_sch (KiCad schematic)
At the start: 21 parts, among them Q1 IRLML6246TRPBF, U1 STM32F405OGYx, U2 STULPI01B, Y1 NX3225GA-10.000M-STD-CRG-2, Y3 FX135A-327

Commit message: MCU_V3_SCH added
Parts:
- removed D1, D2: 1SS417CT,L3F, 1SS417CTL3F, symbol SamacSys_Parts:1SS417CT,L3F
- added C21, C22, C23, C24: GRM155Z71A105KE01J, CAPC1005X55N, symbol SamacSys_Parts:GRM155Z71A105KE01J
- added D1: BAT54S, Package_TO_SOT_SMD:SOT-23, symbol Diode:BAT54S
- added J1: M50-3530242, HDRV2W40P0X127_1X2_254X210X420P, symbol SamacSys_Parts:M50-3530242
- added J2: M50-3530342, HDRV3W40P0X127_1X3_381X210X430P, symbol SamacSys_Parts:M50-3530342
- added R11, R12: ERJ-3EKF1002V, ERJ3EK_(0603), symbol SamacSys_Parts:ERJ-3EKF1002V
- added R21, R22, R24, R25, R26, R27, R28: RK73Z1ETTP, RESC1005X40N, symbol SamacSys_Parts:RK73Z1ETTP
- added R23: ERA2AED123X, ERA2AED122X, symbol SamacSys_Parts:ERA2AED123X
- added R4: CPF0603F100KC1, RESC1608X55N, symbol SamacSys_Parts:CPF0603F100KC1
- renumbered Y1 to Y11, Y3 to Y12
Connections:
- net +3.3: now also H1.1, U2.B2 (VDVIO), U2.B3 (VDVIO), U2.B5 (VDVIO), U2.F3 (VBAT), C23.1, C24.1, D1.2, R11.2, R12.2; no longer H1.2, U2.C4 (~{RESET})
- net +5: now also H1.2; no longer H1.1
- net B1: now also R11.1
- net B2: now also R12.1
- net B4: now also U1.J8 (PA7)
- net GND: now also U2.E2 (VB_REF_FAULT), C21.2, C22.2, C23.2, C24.2, D1.1, J1.2, J2.3, R23.2, R24.1, R4.2; no longer U2.C3 (~{CS}/PWRDN)
- net M1_D1: now also R22.1, R26.1, R28.1; no longer U1.C1 (PA11)
- net M1_D2: now also R21.1, R25.1, R27.1; no longer U1.C2 (PA12)
- net M1_D3: now also U1.G5 (PE13)
- net M1_D4: now also U1.H8 (PA6)
- net M1_D5: now also U1.F5 (PE14)
- net M1_D6: now also U1.G4 (PE15)
- net M1_D7: now also U1.F3 (PC6)
- net M2_D1: now also U1.F8 (PA1)
- net M2_D10: now also U1.G2 (PD12)
- net M2_D2: now also U1.J10 (PA2)
- net M2_D3: now also U1.B5 (PD6)
- net M2_D4: now also U1.A5 (PD7)
- net M2_D5: now also U1.D1 (PA8)
- net M2_D6: now also U1.H2 (PD8)
- net M2_D7: now also U1.H3 (PD9)
- net M2_D8: now also U1.G3 (PD10)
- net M2_D9: now also U1.G1 (PD11)
- net M3_D1: now also U1.D5 (PC10)
- net M3_D2: now also U1.C4 (PC11)
- net M3_D7: now also U1.H1 (PB15)
- net M4_D3: now also U1.J9 (PA4)
- net M4_D4: now also U1.C10 (PA0)
- net M4_D6: now also U1.E2 (PC8)
- net M4_D7: now also U1.J2 (PB14)
- net MCU_BOOT0: now also D1.3, R4.1
- net P0_D3: now also U1.E1 (PC7)
- net SW_CLK: now also J2.2
- net SW_IO: now also J2.1
- net VBAT: now also J1.1
- net at U2.C1 (DM): now also R26.2
- net at U2.C2 (RREF): now also R23.1
- net at U2.D1 (DP): now also R25.2
- net at U2.D3 (ID): now also R24.2
- net at U2.E3 (3V3V): now also C22.1
- net at U2.E6 (1V2V): now also C21.1
- net PC12: now reaches U1.A3 (PC12)
- net PC12: now also R22.2
- net PD2: now reaches U1.B4 (PD2)
- net PD2: now also R21.2
- net ULPI_RST: now reaches U1.F1 (PD15)
- net ULPI_RST: now also U2.C4 (~{RESET})
- net ULPI_PWRDN: now reaches U1.F2 (PD14)
- net ULPI_PWRDN: now also U2.C3 (~{CS}/PWRDN)
- new net PA11: R28.2, U1.C1 (PA11)
- new net PA12: R27.2, U1.C2 (PA12)
Other:
- moved on the sheet: C101, C102, C103, C11, C14, H1, R1

Commit message: MCU_V3 draft added
Parts:
- removed C101: GMD155R71C104KA11D, CAPC1005X55N, symbol SamacSys_Parts:GMD155R71C104KA11D
Connections:
- net GND: now also J1.1, J2.1; no longer J1.2, J2.3
- net SW_IO: now also J2.3; no longer J2.1
- net VBAT: now also J1.2; no longer J1.1

Commit message: MCU_V3 fix3
Parts:
- added C104: GMD155R71C104KA11D, CAPC1005X55N, symbol SamacSys_Parts:GMD155R71C104KA11D
Connections:
- net +3.3: now also C104.2
- net GND: now also C104.1
Changed lines of the file:
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@@
     (stroke (width 0) (type default) (color 0 0 0 0))
   )
+  (wire (pts (xy 216.6112 237.7186) (xy 219.7862 237.7186))
+    (stroke (width 0) (type default) (color 0 0 0 0))
+  )
   (wire (pts (xy 58.42 260.985) (xy 58.42 264.795))
     (stroke (width 0) (type default) (color 0 0 0 0))
@@
     (stroke (width 0) (type default) (color 0 0 0 0))
   )
+  (wire (pts (xy 216.6112 244.7036) (xy 216.6112 237.7186))
+    (stroke (width 0) (type default) (color 0 0 0 0))
+  )
   (wire (pts (xy 95.885 139.065) (xy 123.19 139.065))
     (stroke (width 0) (type default) (color 0 0 0 0))
@@
     (stroke (width 0) (type default) (color 0 0 0 0))
   )
+  (wire (pts (xy 216.6112 257.4036) (xy 216.6112 265.6586))
+    (stroke (width 0) (type default) (color 0 0 0 0))
+  )
   (wire (pts (xy 148.59 121.285) (xy 153.035 121.285))
     (stroke (width 0) (type default) (color 0 0 0 0))
@@
     (effects (font (size 1.27 1.27)) (justify left bottom))
   )
+  (label "+3.3" (at 219.7862 237.7186 0)
+    (effects (font (size 1.27 1.27)) (justify left bottom))
+  )
   (label "M2_D7" (at 266.7 187.96 0)
     (effects (font (size 1.27 1.27)) (justify left bottom))
@@
     (pin "2")
   )
+  (symbol (lib_id "SamacSys_Parts:GMD155R71C104KA11D") (at 216.6112 257.4036 90) (unit 1)
+    (in_bom yes) (on_board yes) (fields_autoplaced)
+    (property "Reference" "C104" (id 0) (at 221.0562 249.7835 90)
+      (effects (font (size 1.27 1.27)) (justify right))
+    )
+    (property "Value" "GMD155R71C104KA11D" (id 1) (at 221.0562 252.3235 90)
+      (effects (font (size 1.27 1.27)) (justify right))
+    )
+    (property "Footprint" "CAPC1005X55N" (id 2) (at 215.3412 248.5136 0)
+      (effects (font (size 1.27 1.27)) (justify left) hide)
+    )
+    (property "Datasheet" "https://psearch.en.murata.com/capacitor/product/GMD155R71C104KA11%23.html" (id 3) (at 217.8812 248.5136 0)
+      (effects (font (size 1.27 1.27)) (justify left) hide)
+    )
+    (property "Description" "Capacitor L=1.0mm W=0.5mm T=0.5mm" (id 4) (at 220.4212 248.5136 0)
+      (effects (font (size 1.27 1.27)) (justify left) hide)
+    )
+    (property "Height" "0.55" (id 5) (at 222.9612 248.5136 0)
+      (effects (font (size 1.27 1.27)) (justify left) hide)
+    )
+    (property "Manufacturer_Name" "Murata Electronics" (id 6) (at 225.5012 248.5136 0)
+      (effects (font (size 1.27 1.27)) (justify left) hide)
+    )
+    (property "Manufacturer_Part_Number" "GMD155R71C104KA11D" (id 7) (at 228.0412 248.5136 0)
+      (effects (font (size 1.27 1.27)) (justify left) hide)
+    )
+    (property "Mouser Part Number" "81-GMD155R71C104KA1D" (id 8) (at 230.5812 248.5136 0)
+      (effects (font (size 1.27 1.27)) (justify left) hide)
+    )
+    (property "Mouser Price/Stock" "https://www.mouser.co.uk/ProductDetail/Murata-Electronics/GMD155R71C104KA11D?qs=YLLXL5qGyDv0d5NAg9etxw%3D%3D" (id 9) (at 233.1212 248.5136 0)
+      (effects (font (size 1.27 1.27)) (justify left) hide)
+    )
+    (property "Arrow Part Number" "GMD155R71C104KA11D" (id 10) (at 235.6612 248.5136 0)
+      (effects (font (size 1.27 1.27)) (justify left) hide)
+    )
+    (property "Arrow Price/Stock" "https://www.arrow.com/en/products/gmd155r71c104ka11d/murata-manufacturing?region=nac" (id 11) (at 238.2012 248.5136 0)
+      (effects (font (size 1.27 1.27)) (justify left) hide)
+    )
+    (pin "1")
+    (pin "2")
+  )
   (symbol (lib_id "SamacSys_Parts:IRLML6246TRPBF") (at 48.26 52.07 0) (mirror y) (unit 1)
     (in_bom yes) (on_board yes) (fields_autoplaced)
@@
     (pin "3")
   )
+  (symbol (lib_id "power:GND") (at 216.6112 265.6586 0) (unit 1)
+    (in_bom yes) (on_board yes) (fields_autoplaced)
+    (property "Reference" "#PWR0107" (id 0) (at 216.6112 272.0086 0)
+      (effects (font (size 1.27 1.27)) hide)
+    )
+    (property "Value" "GND" (id 1) (at 216.6112 270.7386 0))
+    (property "Footprint" "" (id 2) (at 216.6112 265.6586 0)
+      (effects (font (size 1.27 1.27)) hide)
+    )
+    (property "Datasheet" "" (id 3) (at 216.6112 265.6586 0)
+      (effects (font (size 1.27 1.27)) hide)
+    )
+    (pin "1")
+  )
   (symbol (lib_id "SamacSys_Parts:GCQ1555C1H8R0BB01D") (at 257.175 139.065 270) (unit 1)
     (in_bom yes) (on_board yes)
@@
       (reference "#PWR0106") (unit 1) (value "GND") (footprint "")
     )
+    (path "/941be539-a9c4-4972-ac08-696f9cfd0e0f"
+      (reference "#PWR0107") (unit 1) (value "GND") (footprint "")
+    )
     (path "/16ac6937-ccec-4561-8f39-054357731e4b"
       (reference "#PWR0108") (unit 1) (value "GND") (footprint "")
@@
       (reference "C103") (unit 1) (value "GMD155R71C104KA11D") (footprint "CAPC1005X55N")
     )
+    (path "/2f54137a-7ed9-44ec-97e0-8407748f81f4"
+      (reference "C104") (unit 1) (value "GMD155R71C104KA11D") (footprint "CAPC1005X55N")
+    )
     (path "/aaad3178-1732-4ca7-adc4-40a556e02983"

Commit message: MCU_V3 fix4
Changed lines of the file:
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@@
   (junction (at 380.365 204.47) (diameter 0) (color 0 0 0 0)
   )
+  (junction (at 43.307 245.1862) (diameter 0) (color 0 0 0 0)
+  )
   (junction (at 205.74 155.575) (diameter 0) (color 0 0 0 0)
   )
@@
     (stroke (width 0) (type default) (color 0 0 0 0))
   )
+  (wire (pts (xy 40.6654 245.237) (xy 43.307 245.1862))
+    (stroke (width 0) (type default) (color 0 0 0 0))
+  )
